Commit message: updated code: functioning simulation as in paper

File: simulation/gazebo/catkin_ws/src/auto_fisher/urdf/auto_fisher.urdf (robot description, URDF)
Before this commit: robot auto_fisher, 3 links, 2 joints
Joints:
- joint joint1: limit lower=-3.14 upper=3.14 effort=100 velocity=30 -> lower=-3.14 upper=3.14 effort=400 velocity=0.63; type continuous -> revolute
